Commit message: xacro clean up

File: robots/human_right_arm.xacro (robot description, xacro)
@@ -7,4 +7,5 @@
  	<xacro:property name="l2" value="$(arg l2)" />
  	<xacro:property name="l3" value="$(arg l3)" />
+ 	<property name="M_PI" value="3.141592653589793"/>
 	<link name="base_link"/>
 	<link name="link0"/>
@@ -30,5 +31,5 @@
 	<joint name="q1" type="revolute">
 		<origin xyz="0 0 0" rpy="0 0 0"/>
-		<limit lower="-3.141592653589793" upper="3.141592653589793" effort="1000.0" velocity="3"/>
+		<limit lower="${-M_PI}" upper="${M_PI}" effort="1000.0" velocity="3"/>
 		<parent link="base_link"/>
 		<child link="link0"/>
@@ -36,6 +37,6 @@
 	</joint>
 	<joint name="q2" type="revolute">
-		<origin xyz="0 0 0" rpy="1.5707963267948966 0 1.5707963267948966"/>
-		<limit lower="-3.141592653589793" upper="3.141592653589793" effort="1000.0" velocity="3"/>
+		<origin xyz="0 0 0" rpy="${M_PI/2} 0 ${M_PI/2}"/>
+		<limit lower="${-M_PI}" upper="${M_PI}" effort="1000.0" velocity="3"/>
 		<parent link="link0"/>
 		<child link="link1"/>
@@ -43,6 +44,6 @@
 	</joint>
 	<joint name="q3" type="revolute">
-		<origin xyz="0 0 0" rpy="1.5707963267948966 0 1.5707963267948966"/>
-		<limit lower="-3.141592653589793" upper="3.141592653589793" effort="1000.0" velocity="3"/>
+		<origin xyz="0 0 0" rpy="${M_PI/2} 0 ${M_PI/2}"/>
+		<limit lower="${-M_PI}" upper="${M_PI}" effort="1000.0" velocity="3"/>
 		<parent link="link1"/>
 		<child link="link2"/>
@@ -50,6 +51,6 @@
 	</joint>
 	<joint name="q4" type="revolute">
-		<origin xyz="${-l1} 0 0" rpy="1.5707963267948966 0 3.141592653589793"/>
-		<limit lower="-3.141592653589793" upper="3.141592653589793" effort="1000.0" velocity="3"/>
+		<origin xyz="${-l1} 0 0" rpy="${M_PI/2} 0 ${M_PI}"/>
+		<limit lower="${-M_PI}" upper="${M_PI}" effort="1000.0" velocity="3"/>
 		<parent link="link2"/>
 		<child link="link3"/>
@@ -57,6 +58,6 @@
 	</joint>
 	<joint name="q5" type="revolute">
-		<origin xyz="0 0 0" rpy="-1.5707963267948966 0 1.5707963267948966"/>
-		<limit lower="-3.141592653589793" upper="3.141592653589793" effort="1000.0" velocity="3"/>
+		<origin xyz="0 0 0" rpy="${-M_PI/2} 0 ${M_PI/2}"/>
+		<limit lower="${-M_PI}" upper="${M_PI}" effort="1000.0" velocity="3"/>
 		<parent link="link3"/>
 		<child link="link4"/>
@@ -64,6 +65,6 @@
 	</joint>
 	<joint name="q6" type="revolute">
-		<origin xyz="0 0 ${-l2}" rpy="1.5707963267948966 0 0"/>
-		<limit lower="-3.141592653589793" upper="3.141592653589793" effort="1000.0" velocity="3"/>
+		<origin xyz="0 0 ${-l2}" rpy="${M_PI/2} 0 0"/>
+		<limit lower="${-M_PI}" upper="${M_PI}" effort="1000.0" velocity="3"/>
 		<parent link="link4"/>
 		<child link="link5"/>
@@ -71,6 +72,6 @@
 	</joint>
 	<joint name="q7" type="revolute">
-		<origin xyz="0 0 0" rpy="-1.5707963267948966 0 -1.5707963267948966"/>
-		<limit lower="-3.141592653589793" upper="3.141592653589793" effort="1000.0" velocity="3"/>
+		<origin xyz="0 0 0" rpy="${-M_PI/2} 0 ${-M_PI/2}"/>
+		<limit lower="${-M_PI}" upper="${M_PI}" effort="1000.0" velocity="3"/>
 		<parent link="link5"/>
 		<child link="link6"/>
